File: eda/HHV_2019_SC/HHV_2019_SC.kicad_pcb (KiCad board)
At the start: 2 copper layers, 0 parts

Commit message: Soldering Challenge PCB Complete.
Parts:
- added D1: LED_5mm, alt_bier-fp:LED_D5.0mm, F.Cu at (99.0, 57.5)
- added D2: LED_3mm, alt_bier-fp:LED_D3.0mm, F.Cu at (98.5, 71.5)
- added D3: LED_1206, alt_bier-fp:LED_1206_3216Metric_Pad1.42x1.75mm_HandSolder, F.Cu at (100.0, 77.0)
- added D4: LED_0805, alt_bier-fp:LED_0805_2012Metric_Pad1.15x1.40mm_HandSolder, F.Cu at (99.5, 81.5)
- added D5: LED_RCBG_THT_5mm, alt_bier-fp:LED_D5.0mm-4_RGB, F.Cu at (102.0, 89.5)
- added G***: LOGO, alt_bier-logo:logo-alt_bier-700dpi-13x32mm-back, F.Cu at (114.0, 68.5)
- added J1: Battery_Connector, alt_bier-fp:Pin_Header_Straight_1x02_Pitch2.54mm, F.Cu at (134.0, 66.5)
- added R1: R_THT, alt_bier-fp:R_Axial_DIN0207_L6.3mm_D2.5mm_P7.62mm_Horizontal, F.Cu at (106.0, 63.0)
- added R2: R_THT, alt_bier-fp:R_Axial_DIN0207_L6.3mm_D2.5mm_P7.62mm_Horizontal, F.Cu at (106.0, 66.5)
- added R3: R_1206, alt_bier-fp:R_1206_3216Metric_Pad1.42x1.75mm_HandSolder, F.Cu at (109.0, 77.0)
- added R4: R_0805, alt_bier-fp:R_0805_2012Metric_Pad1.15x1.40mm_HandSolder, F.Cu at (109.5, 81.5)
- added R5: R_THT, alt_bier-fp:R_Axial_DIN0207_L6.3mm_D2.5mm_P7.62mm_Horizontal, F.Cu at (124.5, 74.0)
- added R6: R_THT, alt_bier-fp:R_Axial_DIN0207_L6.3mm_D2.5mm_P7.62mm_Horizontal, F.Cu at (128.0, 74.0)
- added R7: R_THT, alt_bier-fp:R_Axial_DIN0207_L6.3mm_D2.5mm_P7.62mm_Horizontal, F.Cu at (131.5, 74.0)
- added S1: SW_Push_Dual_THT_6mm, alt_bier-fp:SW_PUSH_6mm, F.Cu at (112.5, 91.5)
- added S2: SW_Push_Dual_THT_6mm, alt_bier-fp:SW_PUSH_6mm, F.Cu at (123.0, 91.5)
- added S3: SW_Push_Dual_THT_6mm, alt_bier-fp:SW_PUSH_6mm, F.Cu at (133.5, 91.5)
Routing:
- net GND: track 0.00 -> 100.9 mm
- net POS: track 0.00 -> 89.1 mm
- net Net-(D5-Pad4): track 0.00 -> 42.0 mm
- net Net-(D5-Pad3): track 0.00 -> 29.3 mm
- net Net-(R5-Pad2): track 0.00 -> 20.7 mm
- net Net-(D5-Pad1): track 0.00 -> 16.0 mm
- net Net-(R6-Pad2): track 0.00 -> 14.0 mm
- net Net-(R7-Pad2): track 0.00 -> 12.7 mm
- net Net-(D4-Pad2): track 0.00 -> 7.92 mm
- net Net-(D1-Pad2): track 0.00 -> 6.81 mm
- net Net-(D2-Pad2): track 0.00 -> 6.10 mm
- net Net-(D3-Pad2): track 0.00 -> 6.03 mm
Other:
- board outline added: 48 x 48 mm
- net class Default: trace_width 0.25 -> 0.4
- board text added: "16 Parts in 8 Minutes 200 Points Available Most Points Wins Quality is Tie Breaker"
- board text added: "BSidesDFW 2019 Hardware Hacking Village @alt_bier Soldering Challenge"
- board text added: "J1 10pt R1 5pt R2 5pt R3 15pt R4 20pt R5 5pt R6 5pt R7 5pt S1 5pt S2 5pt S3 5pt D1 10pt D2 10pt D3 30pt D4 40pt D5 25pt"
- board text added: "J1 R1 R2 R3 R4 R5 R6 R7 S1 S2 S3 D1 D2 D3 D4 D5"
- board text added: "Name or Handle"
- board text added: "SCORE"
